Commit message: Fixed issues with the dot arm and lidar urdfs.

File: urdf/dot_arm.urdf (robot description, URDF)
Before this commit: robot dot_arm, 31 links, 30 joints
Links:
- link arm_long_U: geometry collision cylinder length=0.02 radius=0.02; visual mesh filename=package://dot/urdf/meshes/long_U.obj
- link arm_section_1: geometry collision cylinder length=0.05 radius=0.02; visual mesh filename=package://dot/urdf/meshes/section_1.obj
- link arm_section_2: geometry collision cylinder length=0.05 radius=0.02; visual mesh filename=package://dot/urdf/meshes/section_2.obj
- link arm_section_3: geometry collision cylinder length=0.05 radius=0.02; visual mesh filename=package://dot/urdf/meshes/section_3.obj
- link arm_section_4: geometry collision cylinder length=0.06 radius=0.02; visual mesh filename=package://dot/urdf/meshes/section_4.obj
- link arm_section_5: geometry collision cylinder length=0.06 radius=0.02; visual mesh filename=package://dot/urdf/meshes/gripper.obj

File: urdf/dot_lidar.urdf (robot description, URDF)
Before this commit: robot dot, 24 links, 23 joints
Links:
- link lidar_link: geometry collision box size=0.0985 0.0577 0.07; visual mesh filename=package://dot/urdf/stl/rplidar_main.stl scale=0.001 0.001 0.001
