Commit message: Fixed Gazebo launch

File: urdf/dot.urdf (robot description, URDF)
Before this commit: robot dot, 23 links, 22 joints
Links:
- link base_link: geometry collision box size=0.14 0.11 0.07; visual mesh filename=file://$(find dot)/urdf/stl/mainbody.stl scale=0.001 0.001 0.001
- link chassis_front_link: geometry collision box size=0.058 0.11 0.07; visual mesh filename=file://$(find dot)/urdf/stl/frontpart.stl scale=0.001 0.001 0.001
- link chassis_rear_link: geometry collision box size=0.04 0.11 0.07; visual mesh filename=file://$(find dot)/urdf/stl/backpart.stl scale=0.001 0.001 0.001
- link front_left_foot_link: geometry collision box size=0.026 0.020 0.115; visual mesh filename=file://$(find dot)/urdf/stl/lfoot.stl scale=0.001 0.001 0.001
- link front_left_leg_link: geometry collision box size=0.028 0.036 0.12; visual mesh filename=file://$(find dot)/urdf/stl/larm.stl scale=0.001 0.001 0.001
- link front_left_leg_link_cover: geometry visual mesh filename=file://$(find dot)/urdf/stl/larm_cover.stl scale=0.001 0.001 0.001
- link front_left_shoulder_link: geometry collision box size=0.044 0.038 0.07; visual mesh filename=file://$(find dot)/urdf/stl/lshoulder.stl scale=0.001 0.001 0.001
- link front_left_toe_link: geometry collision mesh filename=file://$(find dot)/urdf/stl/foot.stl scale=0.001 0.001 0.001; visual mesh filename=file://$(find dot)/urdf/stl/foot.stl scale=0.001 0.001 0.001
- link front_right_foot_link: geometry collision box size=0.026 0.020 0.115; visual mesh filename=file://$(find dot)/urdf/stl/rfoot.stl scale=0.001 0.001 0.001
- link front_right_leg_link: geometry collision box size=0.028 0.036 0.12; visual mesh filename=file://$(find dot)/urdf/stl/rarm.stl scale=0.001 0.001 0.001
- link front_right_leg_link_cover: geometry visual mesh filename=file://$(find dot)/urdf/stl/rarm_cover.stl scale=0.001 0.001 0.001
- link front_right_shoulder_link: geometry collision box size=0.044 0.038 0.07; visual mesh filename=file://$(find dot)/urdf/stl/rshoulder.stl scale=0.001 0.001 0.001
- link front_right_toe_link: geometry collision mesh filename=file://$(find dot)/urdf/stl/foot.stl scale=0.001 0.001 0.001; visual mesh filename=file://$(find dot)/urdf/stl/foot.stl scale=0.001 0.001 0.001
- link rear_left_foot_link: geometry collision box size=0.026 0.020 0.115; visual mesh filename=file://$(find dot)/urdf/stl/lfoot.stl scale=0.001 0.001 0.001
- link rear_left_leg_link: geometry collision box size=0.028 0.036 0.12; visual mesh filename=file://$(find dot)/urdf/stl/larm.stl scale=0.001 0.001 0.001
- link rear_left_leg_link_cover: geometry visual mesh filename=file://$(find dot)/urdf/stl/larm_cover.stl scale=0.001 0.001 0.001
- link rear_left_shoulder_link: geometry collision box size=0.044 0.038 0.07; visual mesh filename=file://$(find dot)/urdf/stl/lshoulder.stl scale=0.001 0.001 0.001
- link rear_left_toe_link: geometry collision mesh filename=file://$(find dot)/urdf/stl/foot.stl scale=0.001 0.001 0.001; visual mesh filename=file://$(find dot)/urdf/stl/foot.stl scale=0.001 0.001 0.001
- link rear_right_foot_link: geometry collision box size=0.026 0.020 0.115; visual mesh filename=file://$(find dot)/urdf/stl/rfoot.stl scale=0.001 0.001 0.001
- link rear_right_leg_link: geometry collision box size=0.028 0.036 0.12; visual mesh filename=file://$(find dot)/urdf/stl/rarm.stl scale=0.001 0.001 0.001
- link rear_right_leg_link_cover: geometry visual mesh filename=file://$(find dot)/urdf/stl/rarm_cover.stl scale=0.001 0.001 0.001
- link rear_right_shoulder_link: geometry collision box size=0.044 0.038 0.07; visual mesh filename=file://$(find dot)/urdf/stl/rshoulder.stl scale=0.001 0.001 0.001
- link rear_right_toe_link: geometry collision mesh filename=file://$(find dot)/urdf/stl/foot.stl scale=0.001 0.001 0.001; visual mesh filename=file://$(find dot)/urdf/stl/foot.stl scale=0.001 0.001 0.001

File: urdf/dot_arm.urdf (robot description, URDF)
Before this commit: robot dot_arm, 31 links, 30 joints
Links:
- link arm_long_U: geometry collision cylinder length=0.02 radius=0.02; visual mesh filename=file://$(find dot)/urdf/meshes/long_U.obj
- link arm_section_1: geometry collision cylinder length=0.05 radius=0.02; visual mesh filename=file://$(find dot)/urdf/meshes/section_1.obj
- link arm_section_2: geometry collision cylinder length=0.05 radius=0.02; visual mesh filename=file://$(find dot)/urdf/meshes/section_2.obj
- link arm_section_3: geometry collision cylinder length=0.05 radius=0.02; visual mesh filename=file://$(find dot)/urdf/meshes/section_3.obj
- link arm_section_4: geometry collision cylinder length=0.06 radius=0.02; visual mesh filename=file://$(find dot)/urdf/meshes/section_4.obj
- link arm_section_5: geometry collision cylinder length=0.06 radius=0.02; visual mesh filename=file://$(find dot)/urdf/meshes/gripper.obj
- link base_link: geometry collision box size=0.14 0.11 0.07; visual mesh filename=file://$(find dot)/urdf/stl/mainbody.stl scale=0.001 0.001 0.001
- link chassis_front_link: geometry collision box size=0.058 0.11 0.07; visual mesh filename=file://$(find dot)/urdf/stl/frontpart.stl scale=0.001 0.001 0.001
- link chassis_rear_link: geometry collision box size=0.04 0.11 0.07; visual mesh filename=file://$(find dot)/urdf/stl/backpart.stl scale=0.001 0.001 0.001
- link front_left_foot_link: geometry collision box size=0.026 0.020 0.115; visual mesh filename=file://$(find dot)/urdf/stl/lfoot.stl scale=0.001 0.001 0.001
- link front_left_leg_link: geometry collision box size=0.028 0.036 0.12; visual mesh filename=file://$(find dot)/urdf/stl/larm.stl scale=0.001 0.001 0.001
- link front_left_leg_link_cover: geometry visual mesh filename=file://$(find dot)/urdf/stl/larm_cover.stl scale=0.001 0.001 0.001
- link front_left_shoulder_link: geometry collision box size=0.044 0.038 0.07; visual mesh filename=file://$(find dot)/urdf/stl/lshoulder.stl scale=0.001 0.001 0.001
- link front_left_toe_link: geometry collision mesh filename=file://$(find dot)/urdf/stl/foot.stl scale=0.001 0.001 0.001; visual mesh filename=file://$(find dot)/urdf/stl/foot.stl scale=0.001 0.001 0.001
- link front_right_foot_link: geometry collision box size=0.026 0.020 0.115; visual mesh filename=file://$(find dot)/urdf/stl/rfoot.stl scale=0.001 0.001 0.001
- link front_right_leg_link: geometry collision box size=0.028 0.036 0.12; visual mesh filename=file://$(find dot)/urdf/stl/rarm.stl scale=0.001 0.001 0.001
- link front_right_leg_link_cover: geometry visual mesh filename=file://$(find dot)/urdf/stl/rarm_cover.stl scale=0.001 0.001 0.001
- link front_right_shoulder_link: geometry collision box size=0.044 0.038 0.07; visual mesh filename=file://$(find dot)/urdf/stl/rshoulder.stl scale=0.001 0.001 0.001
- link front_right_toe_link: geometry collision mesh filename=file://$(find dot)/urdf/stl/foot.stl scale=0.001 0.001 0.001; visual mesh filename=file://$(find dot)/urdf/stl/foot.stl scale=0.001 0.001 0.001
- link rear_left_foot_link: geometry collision box size=0.026 0.020 0.115; visual mesh filename=file://$(find dot)/urdf/stl/lfoot.stl scale=0.001 0.001 0.001
- link rear_left_leg_link: geometry collision box size=0.028 0.036 0.12; visual mesh filename=file://$(find dot)/urdf/stl/larm.stl scale=0.001 0.001 0.001
- link rear_left_leg_link_cover: geometry visual mesh filename=file://$(find dot)/urdf/stl/larm_cover.stl scale=0.001 0.001 0.001
- link rear_left_shoulder_link: geometry collision box size=0.044 0.038 0.07; visual mesh filename=file://$(find dot)/urdf/stl/lshoulder.stl scale=0.001 0.001 0.001
- link rear_left_toe_link: geometry collision mesh filename=file://$(find dot)/urdf/stl/foot.stl scale=0.001 0.001 0.001; visual mesh filename=file://$(find dot)/urdf/stl/foot.stl scale=0.001 0.001 0.001
- link rear_right_foot_link: geometry collision box size=0.026 0.020 0.115; visual mesh filename=file://$(find dot)/urdf/stl/rfoot.stl scale=0.001 0.001 0.001
- link rear_right_leg_link: geometry collision box size=0.028 0.036 0.12; visual mesh filename=file://$(find dot)/urdf/stl/rarm.stl scale=0.001 0.001 0.001
- link rear_right_leg_link_cover: geometry visual mesh filename=file://$(find dot)/urdf/stl/rarm_cover.stl scale=0.001 0.001 0.001
- link rear_right_shoulder_link: geometry collision box size=0.044 0.038 0.07; visual mesh filename=file://$(find dot)/urdf/stl/rshoulder.stl scale=0.001 0.001 0.001
- link rear_right_toe_link: geometry collision mesh filename=file://$(find dot)/urdf/stl/foot.stl scale=0.001 0.001 0.001; visual mesh filename=file://$(find dot)/urdf/stl/foot.stl scale=0.001 0.001 0.001

File: urdf/dot_lidar.urdf (robot description, URDF)
Before this commit: robot dot, 24 links, 23 joints
Links:
- link base_link: geometry collision box size=0.14 0.11 0.07; visual mesh filename=file://$(find dot)/urdf/stl/mainbody.stl scale=0.001 0.001 0.001
- link chassis_front_link: geometry collision box size=0.058 0.11 0.07; visual mesh filename=file://$(find dot)/urdf/stl/frontpart.stl scale=0.001 0.001 0.001
- link chassis_rear_link: geometry collision box size=0.04 0.11 0.07; visual mesh filename=file://$(find dot)/urdf/stl/backpart.stl scale=0.001 0.001 0.001
- link front_left_foot_link: geometry collision box size=0.026 0.020 0.115; visual mesh filename=file://$(find dot)/urdf/stl/lfoot.stl scale=0.001 0.001 0.001
- link front_left_leg_link: geometry collision box size=0.028 0.036 0.12; visual mesh filename=file://$(find dot)/urdf/stl/larm.stl scale=0.001 0.001 0.001
- link front_left_leg_link_cover: geometry visual mesh filename=file://$(find dot)/urdf/stl/larm_cover.stl scale=0.001 0.001 0.001
- link front_left_shoulder_link: geometry collision box size=0.044 0.038 0.07; visual mesh filename=file://$(find dot)/urdf/stl/lshoulder.stl scale=0.001 0.001 0.001
- link front_left_toe_link: geometry collision mesh filename=file://$(find dot)/urdf/stl/foot.stl scale=0.001 0.001 0.001; visual mesh filename=file://$(find dot)/urdf/stl/foot.stl scale=0.001 0.001 0.001
- link front_right_foot_link: geometry collision box size=0.026 0.020 0.115; visual mesh filename=file://$(find dot)/urdf/stl/rfoot.stl scale=0.001 0.001 0.001
- link front_right_leg_link: geometry collision box size=0.028 0.036 0.12; visual mesh filename=file://$(find dot)/urdf/stl/rarm.stl scale=0.001 0.001 0.001
- link front_right_leg_link_cover: geometry visual mesh filename=file://$(find dot)/urdf/stl/rarm_cover.stl scale=0.001 0.001 0.001
- link front_right_shoulder_link: geometry collision box size=0.044 0.038 0.07; visual mesh filename=file://$(find dot)/urdf/stl/rshoulder.stl scale=0.001 0.001 0.001
- link front_right_toe_link: geometry collision mesh filename=file://$(find dot)/urdf/stl/foot.stl scale=0.001 0.001 0.001; visual mesh filename=file://$(find dot)/urdf/stl/foot.stl scale=0.001 0.001 0.001
- link lidar_link: geometry collision box size=0.0985 0.0577 0.07; visual mesh filename=file://$(find dot)/urdf/stl/rplidar_main.stl scale=0.001 0.001 0.001
- link rear_left_foot_link: geometry collision box size=0.026 0.020 0.115; visual mesh filename=file://$(find dot)/urdf/stl/lfoot.stl scale=0.001 0.001 0.001
- link rear_left_leg_link: geometry collision box size=0.028 0.036 0.12; visual mesh filename=file://$(find dot)/urdf/stl/larm.stl scale=0.001 0.001 0.001
- link rear_left_leg_link_cover: geometry visual mesh filename=file://$(find dot)/urdf/stl/larm_cover.stl scale=0.001 0.001 0.001
- link rear_left_shoulder_link: geometry collision box size=0.044 0.038 0.07; visual mesh filename=file://$(find dot)/urdf/stl/lshoulder.stl scale=0.001 0.001 0.001
- link rear_left_toe_link: geometry collision mesh filename=file://$(find dot)/urdf/stl/foot.stl scale=0.001 0.001 0.001; visual mesh filename=file://$(find dot)/urdf/stl/foot.stl scale=0.001 0.001 0.001
- link rear_right_foot_link: geometry collision box size=0.026 0.020 0.115; visual mesh filename=file://$(find dot)/urdf/stl/rfoot.stl scale=0.001 0.001 0.001
- link rear_right_leg_link: geometry collision box size=0.028 0.036 0.12; visual mesh filename=file://$(find dot)/urdf/stl/rarm.stl scale=0.001 0.001 0.001
- link rear_right_leg_link_cover: geometry visual mesh filename=file://$(find dot)/urdf/stl/rarm_cover.stl scale=0.001 0.001 0.001
- link rear_right_shoulder_link: geometry collision box size=0.044 0.038 0.07; visual mesh filename=file://$(find dot)/urdf/stl/rshoulder.stl scale=0.001 0.001 0.001
- link rear_right_toe_link: geometry collision mesh filename=file://$(find dot)/urdf/stl/foot.stl scale=0.001 0.001 0.001; visual mesh filename=file://$(find dot)/urdf/stl/foot.stl scale=0.001 0.001 0.001
