Commit message: Changed File structure

File: dot_description/urdf/dot.urdf (robot description, URDF)
Before this commit: robot dot_arm, 31 links, 30 joints
Links:
- removed link arm_fixed_tip
- removed link arm_long_U
- removed link arm_moving_tip
- removed link arm_section_1
- removed link arm_section_2
- removed link arm_section_3
- removed link arm_section_4
- removed link arm_section_5
- link base_link: geometry collision box size=0.14 0.11 0.07; visual mesh filename=package://dot_description/urdf/stl/mainbody.stl scale=0.001 0.001 0.001
- link chassis_front_link: geometry collision box size=0.058 0.11 0.07; visual mesh filename=package://dot_description/urdf/stl/frontpart.stl scale=0.001 0.001 0.001
- link chassis_rear_link: geometry collision box size=0.04 0.11 0.07; visual mesh filename=package://dot_description/urdf/stl/backpart.stl scale=0.001 0.001 0.001
- link front_left_foot_link: geometry collision box size=0.026 0.020 0.115; visual mesh filename=package://dot_description/urdf/stl/lfoot.stl scale=0.001 0.001 0.001
- link front_left_leg_link: geometry collision box size=0.028 0.036 0.12; visual mesh filename=package://dot_description/urdf/stl/larm.stl scale=0.001 0.001 0.001
- link front_left_leg_link_cover: geometry visual mesh filename=package://dot_description/urdf/stl/larm_cover.stl scale=0.001 0.001 0.001
- link front_left_shoulder_link: geometry collision box size=0.044 0.038 0.07; visual mesh filename=package://dot_description/urdf/stl/lshoulder.stl scale=0.001 0.001 0.001
- link front_left_toe_link: geometry collision mesh filename=package://dot_description/urdf/stl/foot.stl scale=0.001 0.001 0.001; visual mesh filename=package://dot_description/urdf/stl/foot.stl scale=0.001 0.001 0.001
- link front_right_foot_link: geometry collision box size=0.026 0.020 0.115; visual mesh filename=package://dot_description/urdf/stl/rfoot.stl scale=0.001 0.001 0.001
- link front_right_leg_link: geometry collision box size=0.028 0.036 0.12; visual mesh filename=package://dot_description/urdf/stl/rarm.stl scale=0.001 0.001 0.001
- link front_right_leg_link_cover: geometry visual mesh filename=package://dot_description/urdf/stl/rarm_cover.stl scale=0.001 0.001 0.001
- link front_right_shoulder_link: geometry collision box size=0.044 0.038 0.07; visual mesh filename=package://dot_description/urdf/stl/rshoulder.stl scale=0.001 0.001 0.001
- link front_right_toe_link: geometry collision mesh filename=package://dot_description/urdf/stl/foot.stl scale=0.001 0.001 0.001; visual mesh filename=package://dot_description/urdf/stl/foot.stl scale=0.001 0.001 0.001
- link rear_left_foot_link: geometry collision box size=0.026 0.020 0.115; visual mesh filename=package://dot_description/urdf/stl/lfoot.stl scale=0.001 0.001 0.001
- link rear_left_leg_link: geometry collision box size=0.028 0.036 0.12; visual mesh filename=package://dot_description/urdf/stl/larm.stl scale=0.001 0.001 0.001
- link rear_left_leg_link_cover: geometry visual mesh filename=package://dot_description/urdf/stl/larm_cover.stl scale=0.001 0.001 0.001
- link rear_left_shoulder_link: geometry collision box size=0.044 0.038 0.07; visual mesh filename=package://dot_description/urdf/stl/lshoulder.stl scale=0.001 0.001 0.001
- link rear_left_toe_link: geometry collision mesh filename=package://dot_description/urdf/stl/foot.stl scale=0.001 0.001 0.001; visual mesh filename=package://dot_description/urdf/stl/foot.stl scale=0.001 0.001 0.001
- link rear_right_foot_link: geometry collision box size=0.026 0.020 0.115; visual mesh filename=package://dot_description/urdf/stl/rfoot.stl scale=0.001 0.001 0.001
- link rear_right_leg_link: geometry collision box size=0.028 0.036 0.12; visual mesh filename=package://dot_description/urdf/stl/rarm.stl scale=0.001 0.001 0.001
- link rear_right_leg_link_cover: geometry visual mesh filename=package://dot_description/urdf/stl/rarm_cover.stl scale=0.001 0.001 0.001
- link rear_right_shoulder_link: geometry collision box size=0.044 0.038 0.07; visual mesh filename=package://dot_description/urdf/stl/rshoulder.stl scale=0.001 0.001 0.001
- link rear_right_toe_link: geometry collision mesh filename=package://dot_description/urdf/stl/foot.stl scale=0.001 0.001 0.001; visual mesh filename=package://dot_description/urdf/stl/foot.stl scale=0.001 0.001 0.001
Joints:
- removed joint arm_t7f
- removed joint arm_t7m
- removed joint motor_arm_m1
- removed joint motor_arm_m2
- removed joint motor_arm_m3
- removed joint motor_arm_m4
- removed joint motor_arm_m5
- removed joint motor_arm_m6

File: dot_description/urdf/dot_arm.urdf (robot description, URDF)
Before this commit: robot dot, 24 links, 23 joints
Links:
- removed link lidar_link
- added link arm_fixed_tip, mass 0.05
- added link arm_long_U, mass 1.; collision cylinder length=0.02 radius=0.02; visual mesh filename=package://dot_description/urdf/meshes/long_U.obj
- added link arm_moving_tip, mass 0.05
- added link arm_section_1, mass 0.2; collision cylinder length=0.05 radius=0.02; visual mesh filename=package://dot_description/urdf/meshes/section_1.obj
- added link arm_section_2, mass 0.2; collision cylinder length=0.05 radius=0.02; visual mesh filename=package://dot_description/urdf/meshes/section_2.obj
- added link arm_section_3, mass 0.2; collision cylinder length=0.05 radius=0.02; visual mesh filename=package://dot_description/urdf/meshes/section_3.obj
- added link arm_section_4, mass 0.2; collision cylinder length=0.06 radius=0.02; visual mesh filename=package://dot_description/urdf/meshes/section_4.obj
- added link arm_section_5, mass 0.2; collision cylinder length=0.06 radius=0.02; visual mesh filename=package://dot_description/urdf/meshes/gripper.obj
- link base_link: geometry collision box size=0.14 0.11 0.07; visual mesh filename=package://dot_description/urdf/stl/mainbody.stl scale=0.001 0.001 0.001
- link chassis_front_link: geometry collision box size=0.058 0.11 0.07; visual mesh filename=package://dot_description/urdf/stl/frontpart.stl scale=0.001 0.001 0.001
- link chassis_rear_link: geometry collision box size=0.04 0.11 0.07; visual mesh filename=package://dot_description/urdf/stl/backpart.stl scale=0.001 0.001 0.001
- link front_left_foot_link: geometry collision box size=0.026 0.020 0.115; visual mesh filename=package://dot_description/urdf/stl/lfoot.stl scale=0.001 0.001 0.001
- link front_left_leg_link: geometry collision box size=0.028 0.036 0.12; visual mesh filename=package://dot_description/urdf/stl/larm.stl scale=0.001 0.001 0.001
- link front_left_leg_link_cover: geometry visual mesh filename=package://dot_description/urdf/stl/larm_cover.stl scale=0.001 0.001 0.001
- link front_left_shoulder_link: geometry collision box size=0.044 0.038 0.07; visual mesh filename=package://dot_description/urdf/stl/lshoulder.stl scale=0.001 0.001 0.001
- link front_left_toe_link: geometry collision mesh filename=package://dot_description/urdf/stl/foot.stl scale=0.001 0.001 0.001; visual mesh filename=package://dot_description/urdf/stl/foot.stl scale=0.001 0.001 0.001
- link front_right_foot_link: geometry collision box size=0.026 0.020 0.115; visual mesh filename=package://dot_description/urdf/stl/rfoot.stl scale=0.001 0.001 0.001
- link front_right_leg_link: geometry collision box size=0.028 0.036 0.12; visual mesh filename=package://dot_description/urdf/stl/rarm.stl scale=0.001 0.001 0.001
- link front_right_leg_link_cover: geometry visual mesh filename=package://dot_description/urdf/stl/rarm_cover.stl scale=0.001 0.001 0.001
- link front_right_shoulder_link: geometry collision box size=0.044 0.038 0.07; visual mesh filename=package://dot_description/urdf/stl/rshoulder.stl scale=0.001 0.001 0.001
- link front_right_toe_link: geometry collision mesh filename=package://dot_description/urdf/stl/foot.stl scale=0.001 0.001 0.001; visual mesh filename=package://dot_description/urdf/stl/foot.stl scale=0.001 0.001 0.001
- link rear_left_foot_link: geometry collision box size=0.026 0.020 0.115; visual mesh filename=package://dot_description/urdf/stl/lfoot.stl scale=0.001 0.001 0.001
- link rear_left_leg_link: geometry collision box size=0.028 0.036 0.12; visual mesh filename=package://dot_description/urdf/stl/larm.stl scale=0.001 0.001 0.001
- link rear_left_leg_link_cover: geometry visual mesh filename=package://dot_description/urdf/stl/larm_cover.stl scale=0.001 0.001 0.001
- link rear_left_shoulder_link: geometry collision box size=0.044 0.038 0.07; visual mesh filename=package://dot_description/urdf/stl/lshoulder.stl scale=0.001 0.001 0.001
- link rear_left_toe_link: geometry collision mesh filename=package://dot_description/urdf/stl/foot.stl scale=0.001 0.001 0.001; visual mesh filename=package://dot_description/urdf/stl/foot.stl scale=0.001 0.001 0.001
- link rear_right_foot_link: geometry collision box size=0.026 0.020 0.115; visual mesh filename=package://dot_description/urdf/stl/rfoot.stl scale=0.001 0.001 0.001
- link rear_right_leg_link: geometry collision box size=0.028 0.036 0.12; visual mesh filename=package://dot_description/urdf/stl/rarm.stl scale=0.001 0.001 0.001
- link rear_right_leg_link_cover: geometry visual mesh filename=package://dot_description/urdf/stl/rarm_cover.stl scale=0.001 0.001 0.001
- link rear_right_shoulder_link: geometry collision box size=0.044 0.038 0.07; visual mesh filename=package://dot_description/urdf/stl/rshoulder.stl scale=0.001 0.001 0.001
- link rear_right_toe_link: geometry collision mesh filename=package://dot_description/urdf/stl/foot.stl scale=0.001 0.001 0.001; visual mesh filename=package://dot_description/urdf/stl/foot.stl scale=0.001 0.001 0.001
Joints:
- removed joint base_lidar
- added joint arm_t7f: type fixed, parent arm_section_4, child arm_fixed_tip, origin xyz=0 -0.11 0 rpy=-1.5707963267949 0 0
- added joint arm_t7m: type fixed, parent arm_section_5, child arm_moving_tip, origin xyz=0 -0.052 0 rpy=-1.5707963267949 0 0
- added joint motor_arm_m1: type revolute, parent base_link, child arm_long_U, origin xyz=-0.03 0 0.0327993216120967 rpy=0 0 0, axis 0 0 1, limit lower=-1.5 upper=1.5 effort=100.0 velocity=0.7
- added joint motor_arm_m2: type revolute, parent arm_long_U, child arm_section_1, origin xyz=0 0 0.0240006783879033 rpy=0 -1.5707963267949 0, axis 0 0 -1, limit lower=-1.5 upper=1.5 effort=100.0 velocity=0.7
- added joint motor_arm_m3: type revolute, parent arm_section_1, child arm_section_2, origin xyz=0.054 0 0 rpy=0 0 0, axis 0 0 -1, limit lower=-1.5 upper=1.5 effort=100.0 velocity=0.7
- added joint motor_arm_m4: type revolute, parent arm_section_2, child arm_section_3, origin xyz=0.045 0 0 rpy=0 -1.5707963267949 0, axis 0 0 -1, limit lower=-1.5 upper=1.5 effort=100.0 velocity=0.7
- added joint motor_arm_m5: type revolute, parent arm_section_3, child arm_section_4, origin xyz=0 -0.048 0 rpy=0 -1.5707963267949 0, axis 0 0 1, limit lower=-1.5 upper=1.5 effort=100.0 velocity=0.7
- added joint motor_arm_m6: type revolute, parent arm_section_4, child arm_section_5, origin xyz=0 -0.058 0 rpy=0 -1.5707963267949 0, axis 0 0 -1, limit lower=-1.3 upper=.2 effort=100.0 velocity=0.7

File: dot_description/urdf/dot_lidar.urdf (robot description, URDF)
Before this commit: robot dot, 23 links, 22 joints
Links:
- added link lidar_link, mass 0.50; collision box size=0.0985 0.0577 0.07; visual mesh filename=package://dot_description/urdf/stl/rplidar_main.stl scale=0.001 0.001 0.001
- link base_link: geometry collision box size=0.14 0.11 0.07; visual mesh filename=package://dot_description/urdf/stl/mainbody.stl scale=0.001 0.001 0.001
- link chassis_front_link: geometry collision box size=0.058 0.11 0.07; visual mesh filename=package://dot_description/urdf/stl/frontpart.stl scale=0.001 0.001 0.001
- link chassis_rear_link: geometry collision box size=0.04 0.11 0.07; visual mesh filename=package://dot_description/urdf/stl/backpart.stl scale=0.001 0.001 0.001
- link front_left_foot_link: geometry collision box size=0.026 0.020 0.115; visual mesh filename=package://dot_description/urdf/stl/lfoot.stl scale=0.001 0.001 0.001
- link front_left_leg_link: geometry collision box size=0.028 0.036 0.12; visual mesh filename=package://dot_description/urdf/stl/larm.stl scale=0.001 0.001 0.001
- link front_left_leg_link_cover: geometry visual mesh filename=package://dot_description/urdf/stl/larm_cover.stl scale=0.001 0.001 0.001
- link front_left_shoulder_link: geometry collision box size=0.044 0.038 0.07; visual mesh filename=package://dot_description/urdf/stl/lshoulder.stl scale=0.001 0.001 0.001
- link front_left_toe_link: geometry collision mesh filename=package://dot_description/urdf/stl/foot.stl scale=0.001 0.001 0.001; visual mesh filename=package://dot_description/urdf/stl/foot.stl scale=0.001 0.001 0.001
- link front_right_foot_link: geometry collision box size=0.026 0.020 0.115; visual mesh filename=package://dot_description/urdf/stl/rfoot.stl scale=0.001 0.001 0.001
- link front_right_leg_link: geometry collision box size=0.028 0.036 0.12; visual mesh filename=package://dot_description/urdf/stl/rarm.stl scale=0.001 0.001 0.001
- link front_right_leg_link_cover: geometry visual mesh filename=package://dot_description/urdf/stl/rarm_cover.stl scale=0.001 0.001 0.001
- link front_right_shoulder_link: geometry collision box size=0.044 0.038 0.07; visual mesh filename=package://dot_description/urdf/stl/rshoulder.stl scale=0.001 0.001 0.001
- link front_right_toe_link: geometry collision mesh filename=package://dot_description/urdf/stl/foot.stl scale=0.001 0.001 0.001; visual mesh filename=package://dot_description/urdf/stl/foot.stl scale=0.001 0.001 0.001
- link rear_left_foot_link: geometry collision box size=0.026 0.020 0.115; visual mesh filename=package://dot_description/urdf/stl/lfoot.stl scale=0.001 0.001 0.001
- link rear_left_leg_link: geometry collision box size=0.028 0.036 0.12; visual mesh filename=package://dot_description/urdf/stl/larm.stl scale=0.001 0.001 0.001
- link rear_left_leg_link_cover: geometry visual mesh filename=package://dot_description/urdf/stl/larm_cover.stl scale=0.001 0.001 0.001
- link rear_left_shoulder_link: geometry collision box size=0.044 0.038 0.07; visual mesh filename=package://dot_description/urdf/stl/lshoulder.stl scale=0.001 0.001 0.001
- link rear_left_toe_link: geometry collision mesh filename=package://dot_description/urdf/stl/foot.stl scale=0.001 0.001 0.001; visual mesh filename=package://dot_description/urdf/stl/foot.stl scale=0.001 0.001 0.001
- link rear_right_foot_link: geometry collision box size=0.026 0.020 0.115; visual mesh filename=package://dot_description/urdf/stl/rfoot.stl scale=0.001 0.001 0.001
- link rear_right_leg_link: geometry collision box size=0.028 0.036 0.12; visual mesh filename=package://dot_description/urdf/stl/rarm.stl scale=0.001 0.001 0.001
- link rear_right_leg_link_cover: geometry visual mesh filename=package://dot_description/urdf/stl/rarm_cover.stl scale=0.001 0.001 0.001
- link rear_right_shoulder_link: geometry collision box size=0.044 0.038 0.07; visual mesh filename=package://dot_description/urdf/stl/rshoulder.stl scale=0.001 0.001 0.001
- link rear_right_toe_link: geometry collision mesh filename=package://dot_description/urdf/stl/foot.stl scale=0.001 0.001 0.001; visual mesh filename=package://dot_description/urdf/stl/foot.stl scale=0.001 0.001 0.001
Joints:
- added joint base_lidar: type fixed, parent base_link, child lidar_link, origin xyz=0 0 0.035
